File: R7FA8M1AHECFB_v1.kicad_sch (KiCad schematic)
At the start: 101 parts, among them IC101 R7FA8M1AHECFB#AA0, J101 Conn_01x04_Pin, J102 Conn_01x10_Pin, J103 USB_C_Receptacle, J104 Conn_01x05_Pin, J105 Conn_01x06_Pin, J106 Conn_01x06_Pin, J107 Conn_01x04_Pin, J108 Conn_01x04_Pin, J109 5051102296, J110 DM3AT-SF-PEJM5, SW101 SKRPADE010, SW102 SKRPADE010, SW103 SKRPADE010, SW104 SKRPADE010, SW105 SKRPADE010, SW106 SKRPADE010, SW107 SW_Nidec_CAS-120A1, Y101 KC2016Z20.0000C1KX00

Commit message: こみこみーーー
Parts:
- removed J105: Conn_01x06_Pin, Connector_JST:JST_XA_B06B-XASK-1_1x06_P2.50mm_Vertical, symbol libV 1:Conn_01x06_Pin
- removed J108: Conn_01x04_Pin, Connector_JST:JST_XA_B04B-XASK-1_1x04_P2.50mm_Vertical, symbol libV 1:Conn_01x04_Pin
- removed R130: 33, Resistor_SMD:R_0603_1608Metric, symbol libV 1:R
- removed SW101, SW104: SKRPADE010, 00_myFoot_7.0Lib:SKRPADE010_AAL, symbol libV 1:SKRPADE010
- added SW108: SKRPADE010, 00_myFoot_7.0Lib:SKRPADE010_AAL, symbol libV 1:SKRPADE010
- J101, J107: footprint Connector_JST:JST_XA_B04B-XASK-1_1x04_P2.50mm_Vertical -> 00_myFoot_7.0Lib:B04BPASKLFSN
- J102: footprint 00_myFoot_7.0Lib:SAMTEC_FTSH-105-X-X-DV-007-P-X -> 00_myFoot_7.0Lib:CONN_3220-10-0100-00_CNC
- J104: footprint Connector_JST:JST_XA_B05B-XASK-1_1x05_P2.50mm_Vertical -> 00_myFoot_7.0Lib:B05BPASK1
- J106: footprint Connector_JST:JST_XA_B06B-XASK-1_1x06_P2.50mm_Vertical -> 00_myFoot_7.0Lib:B06BPASK1LFSN
- RV102: footprint Connector_JST:JST_XA_B03B-XASK-1_1x03_P2.50mm_Vertical -> 00_myFoot_7.0Lib:B03BPASKLFSN
Connections:
- net GND: now also SW108.3
- net P308_SD_CLK: now also J110.5 (CLK)
- net RESET: now also SW108.2
- no-connect marks 52 -> 53

Commit message: うぎゃああああああああああ
Parts:
- removed D109, D110, D111, D112, D113, D114, D115, D116: LED, LED_SMD:LED_0603_1608Metric, symbol libV 1:LED
- removed R111, R112, R113, R114, R115, R116, R117, R118: 330, Resistor_SMD:R_0603_1608Metric, symbol libV 1:R
Connections:
- no-connect marks 53 -> 61
