File: dengen.kicad_sch (KiCad schematic)
At the start: 14 parts, among them IC201 MAXM17634AMG+T, J201 Conn_01x02_Pin, U201 LDL1117S33R

Commit message: こみこみーーー
Connections:
- net +12V: now also J201.2 (Pin_2); no longer J201.1 (Pin_1)
- net GND: now also J201.1 (Pin_1); no longer J201.2 (Pin_2)
Changed lines of the file:
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@@
   (junction (at 171.45 76.2) (diameter 0) (color 0 0 0 0)
   )
-  (junction (at 64.77 80.01) (diameter 0) (color 0 0 0 0)
-  )
   (junction (at 64.77 72.39) (diameter 0) (color 0 0 0 0)
   )
@@
   )
   (junction (at 115.57 83.82) (diameter 0) (color 0 0 0 0)
+  )
+  (junction (at 64.77 81.28) (diameter 0) (color 0 0 0 0)
   )
   (junction (at 115.57 76.2) (diameter 0) (color 0 0 0 0)
@@
     (stroke (width 0) (type default))
   )
+  (wire (pts (xy 50.8 77.47) (xy 64.77 77.47))
+    (stroke (width 0) (type default))
+  )
   (wire (pts (xy 242.57 86.36) (xy 248.92 86.36))
     (stroke (width 0) (type default))
@@
     (stroke (width 0) (type default))
   )
-  (wire (pts (xy 50.8 74.93) (xy 64.77 74.93))
+  (wire (pts (xy 50.8 74.93) (xy 53.34 74.93))
+    (stroke (width 0) (type default))
+  )
+  (wire (pts (xy 53.34 81.28) (xy 64.77 81.28))
     (stroke (width 0) (type default))
   )
@@
     (stroke (width 0) (type default))
   )
-  (wire (pts (xy 64.77 74.93) (xy 64.77 72.39))
+  (wire (pts (xy 64.77 77.47) (xy 64.77 72.39))
     (stroke (width 0) (type default))
   )
@@
     (stroke (width 0) (type default))
   )
-  (wire (pts (xy 64.77 80.01) (xy 64.77 87.63))
+  (wire (pts (xy 64.77 80.01) (xy 64.77 81.28))
     (stroke (width 0) (type default))
   )
@@
     (stroke (width 0) (type default))
   )
+  (wire (pts (xy 53.34 74.93) (xy 53.34 81.28))
+    (stroke (width 0) (type default))
+  )
   (wire (pts (xy 242.57 97.79) (xy 242.57 91.44))
     (stroke (width 0) (type default))
@@
     (stroke (width 0) (type default))
   )
+  (wire (pts (xy 64.77 81.28) (xy 64.77 87.63))
+    (stroke (width 0) (type default))
+  )
   (wire (pts (xy 138.43 44.45) (xy 138.43 34.29))
     (stroke (width 0) (type default))
@@
     (stroke (width 0) (type default))
   )
-  (wire (pts (xy 50.8 77.47) (xy 64.77 77.47))
-    (stroke (width 0) (type default))
-  )
   (wire (pts (xy 125.73 50.8) (xy 115.57 50.8))
     (stroke (width 0) (type default))
@@
     (stroke (width 0) (type default))
   )
-  (wire (pts (xy 64.77 77.47) (xy 64.77 80.01))
-    (stroke (width 0) (type default))
-  )

Commit message: うぎゃああああああああああ
Parts:
- added D203: 1.5KExxA, Diode_THT:D_A-405_P10.16mm_Horizontal, symbol Diode:1.5KExxA
Connections:
- net +12V: now also D203.1 (A1)
- net GND: now also D203.2 (A2)
Changed lines of the file:
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@@
   (junction (at 115.57 76.2) (diameter 0) (color 0 0 0 0)
   )
+  (junction (at 58.42 81.28) (diameter 0) (color 0 0 0 0)
+  )
   (junction (at 242.57 72.39) (diameter 0) (color 0 0 0 0)
   )
@@
   )
   (junction (at 242.57 86.36) (diameter 0) (color 0 0 0 0)
+  )
+  (junction (at 58.42 72.39) (diameter 0) (color 0 0 0 0)
   )
   (junction (at 151.13 76.2) (diameter 0) (color 0 0 0 0)
@@
     (stroke (width 0) (type default))
   )
-  (wire (pts (xy 50.8 77.47) (xy 64.77 77.47))
+  (wire (pts (xy 50.8 77.47) (xy 55.88 77.47))
     (stroke (width 0) (type default))
   )
@@
     (stroke (width 0) (type default))
   )
+  (wire (pts (xy 58.42 81.28) (xy 64.77 81.28))
+    (stroke (width 0) (type default))
+  )
   (wire (pts (xy 104.14 83.82) (xy 115.57 83.82))
     (stroke (width 0) (type default))
@@
     (stroke (width 0) (type default))
   )
-  (wire (pts (xy 53.34 81.28) (xy 64.77 81.28))
+  (wire (pts (xy 53.34 81.28) (xy 58.42 81.28))
     (stroke (width 0) (type default))
   )
@@
     (stroke (width 0) (type default))
   )
+  (wire (pts (xy 55.88 72.39) (xy 58.42 72.39))
+    (stroke (width 0) (type default))
+  )
   (wire (pts (xy 248.92 93.98) (xy 248.92 97.79))
     (stroke (width 0) (type default))
@@
     (stroke (width 0) (type default))
   )
-  (wire (pts (xy 64.77 77.47) (xy 64.77 72.39))
+  (wire (pts (xy 55.88 77.47) (xy 55.88 72.39))
     (stroke (width 0) (type default))
   )
@@
     (stroke (width 0) (type default))
   )
+  (wire (pts (xy 58.42 72.39) (xy 58.42 73.66))
+    (stroke (width 0) (type default))
+  )
   (wire (pts (xy 115.57 76.2) (xy 115.57 78.74))
     (stroke (width 0) (type default))
@@
   )
   (wire (pts (xy 115.57 50.8) (xy 115.57 60.96))
+    (stroke (width 0) (type default))
+  )
+  (wire (pts (xy 58.42 72.39) (xy 64.77 72.39))
     (stroke (width 0) (type default))
   )
@@
         )
       )
+    )
+  )
+  (symbol (lib_id "Diode:1.5KExxA") (at 58.42 77.47 270) (unit 1)
+    (in_bom yes) (on_board yes) (dnp no) (fields_autoplaced)
+    (property "Reference" "D203" (at 60.96 76.2 90)
+      (effects (font (size 1.27 1.27)) (justify left))
+    )
+    (property "Value" "1.5KExxA" (at 60.96 78.74 90)
+      (effects (font (size 1.27 1.27)) (justify left))
+    )
+    (property "Footprint" "Diode_THT:D_A-405_P10.16mm_Horizontal" (at 53.34 77.47 0)
+      (effects (font (size 1.27 1.27)) hide)
+    )
+    (property "Datasheet" "https://www.vishay.com/docs/88301/15ke.pdf" (at 58.42 76.2 0)
+      (effects (font (size 1.27 1.27)) hide)
+    )
+    (pin "2")
+    (pin "1")
+    (instances
+      (project "R7FA8M1AHECFB_v1"
+        (path "/8e3ca2dd-888b-4e54-abdd-74ad184656fa/0c035284-2691-4377-8775-287ed1c004af"
+          (reference "D203") (unit 1)
+        )
+      )
