File: R7FA8M1AHECFB_v1.kicad_pcb (KiCad board)
At the start: 2 copper layers, 60 x 75 mm, 119 parts, among them IC101 R7FA8M1AHECFB#AA0, IC201 MAXM17634AMG+T, J101 Conn_01x04_Pin, J102 Conn_01x10_Pin, J103 USB_C_Receptacle, J104 Conn_01x05_Pin, J105 Conn_01x06_Pin, J106 Conn_01x06_Pin, J107 Conn_01x04_Pin, J108 Conn_01x04_Pin, J109 5051102296, J110 DM3AT-SF-PEJM5, J201 Conn_01x02_Pin, SW101 SKRPADE010, SW102 SKRPADE010, SW103 SKRPADE010, SW104 SKRPADE010, SW105 SKRPADE010, SW106 SKRPADE010, SW107 SW_Nidec_CAS-120A1, U201 LDL1117S33R, Y101 KC2016Z20.0000C1KX00

Commit message: こみこみーーー
Parts:
- removed J105: Conn_01x06_Pin, Connector_JST:JST_XA_B06B-XASK-1_1x06_P2.50mm_Vertical
- removed J108: Conn_01x04_Pin, Connector_JST:JST_XA_B04B-XASK-1_1x04_P2.50mm_Vertical
- removed SW101, SW104: SKRPADE010, 00_myFoot_7.0Lib:SKRPADE010_AAL
- added SW108: SKRPADE010, 00_myFoot_7.0Lib:SKRPADE010_AAL, F.Cu at (111.6, 94.5)
- C204, R202: moved to F.Cu
- J101, J107: footprint Connector_JST:JST_XA_B04B-XASK-1_1x04_P2.50mm_Vertical -> 00_myFoot_7.0Lib:B04BPASKLFSN
- J102: footprint 00_myFoot_7.0Lib:SAMTEC_FTSH-105-X-X-DV-007-P-X -> 00_myFoot_7.0Lib:CONN_3220-10-0100-00_CNC
- J104: footprint Connector_JST:JST_XA_B05B-XASK-1_1x05_P2.50mm_Vertical -> 00_myFoot_7.0Lib:B05BPASK1
- J106: footprint Connector_JST:JST_XA_B06B-XASK-1_1x06_P2.50mm_Vertical -> 00_myFoot_7.0Lib:B06BPASK1LFSN
- RV102: footprint Connector_JST:JST_XA_B03B-XASK-1_1x03_P2.50mm_Vertical -> 00_myFoot_7.0Lib:B03BPASKLFSN
- moved R108 117.3 mm to (117.2, 145.7)
- moved R111 117.3 mm to (117.2, 153.2)
- moved R118 117.3 mm to (121.2, 145.7)
- moved R128 117.3 mm to (125.2, 145.7)
- moved R112 117.3 mm to (121.2, 130.6)
- moved R115 117.3 mm to (121.2, 138.2)
- moved R122 117.3 mm to (125.2, 130.6)
- moved R107 117.3 mm to (117.2, 143.2)
- moved R109 117.3 mm to (117.2, 148.2)
- moved R110 117.3 mm to (117.2, 150.7)
- moved R113 117.3 mm to (121.2, 133.1)
- moved R114 117.3 mm to (121.2, 135.7)
- moved R116 117.3 mm to (121.2, 140.7)
- moved R117 117.3 mm to (121.2, 143.2)
- moved R119 117.3 mm to (121.2, 148.2)
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Connections:
- J110 pad 5: Net-(J110-CLK) -> /P308_SD_CLK
- J201 pad 1: +12V -> GND
- J201 pad 2: GND -> +12V

Commit message: おんぎゃ
Parts:
- removed R130: 33, Resistor_SMD:R_0603_1608Metric
- R101, R102, R103, R104, R105, R107, R109, R110, R111, R112, R113, R114, R115, R116, R117, R118, R119, R120, R122, R123, R128, R129: moved to B.Cu
- moved R110 33.8 mm to (129.7, 119.3), turned to 90 degrees
- moved R108 33.3 mm to (127.1, 113.9), turned to -90 degrees
- moved R109 30.9 mm to (128.1, 119.3), turned to 90 degrees
- moved R111 29.3 mm to (119.0, 124.0), turned to 90 degrees
- moved R107 25.7 mm to (126.6, 119.3), turned to 90 degrees
- moved R120 24.3 mm to (117.0, 126.7), turned to 180 degrees
- moved R118 23.3 mm to (129.7, 124.0), turned to 90 degrees
- moved R119 22.7 mm to (113.9, 126.7), turned to 180 degrees
- moved R129 22.1 mm to (120.0, 126.7), turned to 180 degrees
- moved R117 20.4 mm to (128.1, 124.0), turned to 90 degrees
- moved R128 19.3 mm to (117.0, 128.3), turned to 180 degrees
- moved R116 17.6 mm to (126.6, 124.0), turned to 90 degrees
- moved R115 14.7 mm to (125.1, 124.0), turned to 90 degrees
- moved R101 12.7 mm to (119.0, 119.3)
- moved R102 12.7 mm to (120.5, 119.3)
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Routing:
- net +3.3V: track 0.00 -> 31.0 mm
- net Net-(D117-A): track 0.00 -> 23.6 mm, vias 0 -> 3
- net /VCL_1: track 0.00 -> 16.0 mm, vias 0 -> 1
- net /P815_USB_DM: track 0.00 -> 13.7 mm
- net /P814_USB_DP: track 0.00 -> 13.6 mm
- net /P407_USB_VBUS: track 0.00 -> 9.37 mm
- net +5V: track 0.00 -> 9.28 mm, vias 0 -> 2
- net /VLO: track 0.00 -> 7.06 mm, vias 0 -> 1
- net Net-(IC101-XCIN): track 0.00 -> 2.62 mm
- net Net-(J103-CC2): track 0.00 -> 2.58 mm
- net Net-(J103-CC1): track 0.00 -> 2.44 mm
- net Net-(IC201-BST): track 0.00 -> 2.21 mm
- net /EXTAL: track 0.00 -> 2.01 mm
Other:
- copper layers 2 -> 4

Commit message: うぎゃああああああああああ
Parts:
- removed D109, D110, D111, D112, D113, D114, D115, D116: LED, LED_SMD:LED_0603_1608Metric
- removed R111, R112, R113, R114, R115, R116, R117, R118: 330, Resistor_SMD:R_0603_1608Metric
- added D203: 1.5KExxA, Diode_THT:D_A-405_P10.16mm_Horizontal, B.Cu at (161.1, 101.0)
- moved LED101 15.9 mm to (127.1, 125.7)
- moved R119 12.9 mm to (126.7, 125.2), turned to -90 degrees
- moved R128 11.7 mm to (128.3, 125.2), turned to -90 degrees
- moved R122 11.7 mm to (125.2, 125.2), turned to -90 degrees
- moved LED102 8.38 mm to (122.5, 125.7)
- moved R120 5.45 mm to (122.2, 125.1), turned to -90 degrees
- moved R129 4.02 mm to (123.7, 125.1), turned to -90 degrees
- moved R123 3.18 mm to (120.7, 125.2), turned to -90 degrees
- turned SW103 to -90 degrees
Routing:
- net +3.3V: track 31.0 -> 345.3 mm, vias 0 -> 34
- net +5V: track 9.28 -> 97.6 mm, vias 2 -> 9
- net /P400_SCL: track 0.00 -> 83.9 mm, vias 0 -> 1
- net /P415_ENC_B: track 0.00 -> 82.5 mm, vias 0 -> 1
- net /P414_ENC_A: track 0.00 -> 82.2 mm, vias 0 -> 1
- net /P401_SDA: track 0.00 -> 78.8 mm, vias 0 -> 1
- net /P702_FLED1_B: track 0.00 -> 78.4 mm, vias 0 -> 2
- net /P701_FLED1_G: track 0.00 -> 76.0 mm, vias 0 -> 2
- net /P700_FLED1_R: track 0.00 -> 73.3 mm, vias 0 -> 2
- net /P709_LED4: track 0.00 -> 73.3 mm, vias 0 -> 2
- net /P710_LED3: track 0.00 -> 70.2 mm, vias 0 -> 2
- net /P711_LED2: track 0.00 -> 67.7 mm, vias 0 -> 2
- net GND: track 0.00 -> 66.3 mm, vias 0 -> 107
- net /VCL_1: track 16.0 -> 81.7 mm, vias 1 -> 4
- net /P703_FLED2_R: track 0.00 -> 65.7 mm, vias 0 -> 3
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- added copper zone on F.Cu, net +12V
- added copper zone on In1.Cu, net +3.3V
- added copper zone on In2.Cu, net +3.3V
- added copper zone on F.Cu, net +5V
- added copper zone on B.Cu, net GND
- added copper zone on F.Cu, net GND

Commit message: こみこみーーー
Routing:
- net /P708_LED5: track 61.5 -> 58.7 mm
- net /P709_LED4: track 73.3 -> 70.4 mm
- net /P413_LED6: track 59.1 -> 56.8 mm
- net /P412_LED7: track 57.3 -> 55.0 mm
- net /P710_LED3: track 70.2 -> 67.9 mm
- net /P711_LED2: track 67.7 -> 65.4 mm
- net /P712_LED1: track 65.4 -> 63.1 mm
- net /P704_FLED2_G: track 64.0 -> 61.9 mm
- net /P713_LED0: track 62.8 -> 60.7 mm
- net /P702_FLED1_B: track 78.4 -> 76.4 mm
- net /P701_FLED1_G: track 76.0 -> 74.0 mm
- net /P700_FLED1_R: track 73.3 -> 71.2 mm
- net /P703_FLED2_R: track 65.7 -> 64.2 mm
- net /P705_FLED2_B: track 61.0 -> 59.5 mm
- net /P610_SPI0_SCK: track 46.3 -> 47.7 mm
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
Commit message: おおおおおおお
Routing:
- net +3.3V: track 345.3 -> 104.7 mm, vias 34 -> 52
- net GND: vias 117 -> 119
- added copper zone on F.Cu, net +3.3V

Commit message: おおおおおおおおお
Routing:
- net +3.3V: track 104.7 -> 110.7 mm
- net /P414_ENC_A: track 82.3 -> 82.2 mm, vias 2 -> 1

Commit message: 配線微調整
Routing:
- net /P610_SPI0_SCK: track 47.7 -> 45.3 mm
- net /P400_SCL: track 83.2 -> 81.3 mm
- net /P602_RR_SR: track 31.1 -> 30.1 mm
- net /P114_SPI0_CS0: track 42.8 -> 43.5 mm
- net /P115_SPI0_MOSI: track 39.9 -> 40.6 mm
- net /P611_RL_PHASE: track 40.4 -> 39.6 mm
- net /P705_FLED2_B: track 59.5 -> 60.1 mm
- net /P709_LED4: track 70.4 -> 70.9 mm
- net /P710_LED3: track 67.9 -> 68.4 mm
- net /P712_LED1: track 63.1 -> 63.7 mm
- net /P711_LED2: track 65.4 -> 65.9 mm
- net /P614_ST_PHASE: track 40.1 -> 39.6 mm
- net +3.3V: vias 52 -> 53
